File: PCB/kicad/Alice_PCB.kicad_pcb (KiCad board)
At the start: 2 copper layers, 337.5 x 123.1 mm, 172 parts

Commit message: Fixed USB port positioning
fixed the USB port position to fit other alice style cases, as well as changed USB from bottom to top mount
Parts:
- USB1: moved to F.Cu
- moved R_USB1 31.4 mm to (139.7, 44.3), turned to 180 degrees
- moved R_USB2 31.4 mm to (149.2, 44.3), turned to 0 degrees
- moved USB1 30.1 mm to (144.1, 34.3), turned to 180 degrees
- moved C_Shield1 29.9 mm to (151.9, 44.6)
- moved R_Shield1 29.9 mm to (151.9, 43.6)
- moved D_ESD1 29.9 mm to (144.1, 46.6)
- moved F1 29.9 mm to (147.3, 48.5)
- moved R_LED3 29.9 mm to (-22.6, 134.7)
- moved C_VDD1 29.9 mm to (143.5, 105.4)
- moved C_VDDA2 29.9 mm to (136.7, 111.4)
- moved C_VDDIO1 29.9 mm to (141.1, 96.7)
- moved D_LED_Caps1 29.9 mm to (-22.6, 127.9)
- moved D_LED_Layer1 29.9 mm to (-22.6, 136.9)
- moved D_LED_Scroll1 29.9 mm to (-22.6, 132.4)
- moved D_SW_5 29.9 mm to (114.2, 64.3)
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Routing:
- net Net-(USB1-Pad10): track 5.71 -> 4.45 mm, vias 2 -> 1
- net GNDPWR: track 23.0 -> 24.2 mm
- net D+: track 63.0 -> 63.7 mm, vias 0 -> 3
- net D-: track 62.0 -> 62.5 mm, vias 0 -> 1
- net VCC: track 15.9 -> 15.4 mm, vias 0 -> 1
- net GND: track 109.7 -> 109.3 mm, vias 12 -> 14
- net Net-(USB1-Pad4): track 4.85 -> 5.18 mm, vias 0 -> 1
Other:
- outline, holes or cut-outs redrawn
